File: PCB/AmidalaShield.kicad_sch (KiCad schematic)
At the start: 1 part

Commit message: refactor: Update PCB with power jumper
This adds a jumper to connect the digital and analog pins to either 3.3v or 5v depending on the jumper position.
Parts:
- ESP32-S3: now left out of the parts list
Changed lines of the file:
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@@
 		(unit 1)
 		(exclude_from_sim no)
-		(in_bom yes)
+		(in_bom no)
 		(on_board yes)
 		(dnp no)
