File: PCB/spi.kicad_sch (KiCad schematic)
At the start: 14 parts, among them J3 Micro_SD_Card

Commit message: refactor: Update PCB with power jumper
This adds a jumper to connect the digital and analog pins to either 3.3v or 5v depending on the jumper position.
Parts:
- SPI1, XBee3: now left out of the parts list
Changed lines of the file:
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@@
 		(unit 1)
 		(exclude_from_sim no)
-		(in_bom yes)
+		(in_bom no)
 		(on_board yes)
 		(dnp no)
@@
 		(unit 1)
 		(exclude_from_sim no)
-		(in_bom yes)
-		(on_board yes)
-		(dnp no)
+		(in_bom no)
+		(on_board yes)
+		(dnp no)
