File: PCB/AmidalaShield.kicad_pcb (KiCad board)
At the start: 4 copper layers, 99.9 x 74.9 mm, 40 parts, among them J1 Screw_Terminal_01x02, J3 Micro_SD_Card

Commit message: Port Amidala Shield hardware design to Stackup (#232)
Replace the KiCad schematics with a Stackup KDL design (PCB/stackup/)
backed by the pinned Stackup parts library, plus project parts for the
ESP32-S3-DevKitC-1, Hirose microSD socket, screw terminal and 3-way
jumper. The port is 1:1: same parts, designators, footprints and net
names, and every connected pad lands on the same net as before.

Adopt the existing routed PCB by giving each footprint its Stackup
identity, then sync it with the Stackup KiCad plugin. Copper, footprint
positions, silkscreen, mask and paste are unchanged; the sync only adds
Stackup fields, adds units to R/C values, and drops the placeholder nets
on no-connect pads.

Add a Cargo-locked Stackup 0.2.0 CLI and a CI job that checks the design
and fails if syncing would change the committed PCB.

Co-authored-by: Claude Opus 5.5 <noreply@anthropic.com>
Parts:
- C1, C2, C3: value 100n -> 100nF
- C4, C7: value 10u -> 10µF
- C5: value 1u -> 1µF
- C6: value 8.2p -> 8.2pF
- R1, R2, R3, R5: value 10k -> 10kΩ
Connections:
- ESP32-S3 pad 14: unconnected-(ESP32-S3-GPIO46-Pad14) -> (no net)
- ESP32-S3 pad 25: unconnected-(ESP32-S3-GPIO19/USB_D--Pad25) -> (no net)
- ESP32-S3 pad 26: unconnected-(ESP32-S3-GPIO20/USB_D+-Pad26) -> (no net)
- ESP32-S3 pad 29: unconnected-(ESP32-S3-GPIO48-Pad29) -> (no net)
- ESP32-S3 pad 3: unconnected-(ESP32-S3-CHIP_PU-Pad3) -> (no net)
- ESP32-S3 pad 30: unconnected-(ESP32-S3-GPIO45-Pad30) -> (no net)
- ESP32-S3 pad 31: unconnected-(ESP32-S3-GPIO0-Pad31) -> (no net)
- ESP32-S3 pad 32: unconnected-(ESP32-S3-GPIO35-Pad32)_1 -> (no net)
- ESP32-S3 pad 33: unconnected-(ESP32-S3-GPIO36-Pad33) -> (no net)
- ESP32-S3 pad 34: unconnected-(ESP32-S3-GPIO37-Pad34)_1 -> (no net)
- J3 pad 1: unconnected-(J3-DAT2-Pad1) -> (no net)
- J3 pad 10: unconnected-(J3-DET_A-Pad10) -> (no net)
- J3 pad 8: unconnected-(J3-DAT1-Pad8) -> (no net)
- J3 pad 9: unconnected-(J3-DET_B-Pad9) -> (no net)
- XBee3 pad 12: unconnected-(XBee3-~{CTS}/DIO7-Pad12) -> (no net)
- XBee3 pad 14: unconnected-(XBee3-[RESERVED]_2-Pad14) -> (no net)
- XBee3 pad 15: unconnected-(XBee3-ASSOCIATE/DIO5-Pad15) -> (no net)
- XBee3 pad 16: unconnected-(XBee3-~{RTS}/DIO6-Pad16) -> (no net)
- XBee3 pad 2: unconnected-(XBee3-DOUT/DIO13-Pad2) -> (no net)
- XBee3 pad 20: unconnected-(XBee3-AD0_/DIO0-Pad20) -> (no net)
- XBee3 pad 3: unconnected-(XBee3-DIN/~{CONFIG}/DIO14-Pad3) -> (no net)
- XBee3 pad 6: unconnected-(XBee3-RSSI_PWM/DIO10-Pad6) -> (no net)
- XBee3 pad 7: unconnected-(XBee3-PWM1/DIO11-Pad7) -> (no net)
- XBee3 pad 8: unconnected-(XBee3-[RESERVED]_1-Pad8) -> (no net)
